Commit message: plot link com

File: bi_urdf/urdf/bi_urdf(1).urdf (robot description, URDF)
Before this commit: robot bi_urdf, 16 links, 15 joints
Links:
- link lw_Link: mass 0.280 -> 0.0
- link rw_Link: mass 0.280 -> 0.0
Joints:
- joint L_base2hip: limit (none) -> lower=0.0 upper=0.0 effort=0.0 velocity=0.0; type fixed -> revolute
- joint L_hip2thigh: child lu_Link -> lll_Link; limit (none) -> lower=0.0 upper=1.57 effort=23.7 velocity=30.0; origin xyz=0 0.0577075781855487 0 rpy=0 1.2164473167519347 0 -> xyz=0.0532497748906447 0.0144424855132758 0 rpy=0 0 0; parent lll_Link -> ll_Link; type fixed -> revolute
- joint L_thigh2calf: limit (none) -> lower=-2.61 upper=0.0 effort=23.7 velocity=30.0; origin xyz=0 0 -0.215 rpy=0 -2.139803613507067 0 -> xyz=0 0 -0.215 rpy=0 0 0; type fixed -> revolute
- joint L_thigh_fix: child lll_Link -> lu_Link; origin xyz=0.0532497748906447 0.0144424855132758 0 rpy=0 0 0 -> xyz=0 0.0577075781855487 0 rpy=0 0 0; parent ll_Link -> lll_Link
- joint R_base2hip: limit (none) -> lower=0.0 upper=0.0 effort=0.0 velocity=0.0; type fixed -> revolute
- joint R_hip2thigh: child ru_Link -> rrr_Link; limit (none) -> lower=0.0 upper=1.57 effort=23.7 velocity=30.0; origin xyz=0 -0.0577075781855466 0 rpy=0 1.2164473167519347 0 -> xyz=0.0532497748906444 -0.0144424855132765 0 rpy=0 0 0; parent rrr_Link -> rr_Link; type fixed -> revolute
- joint R_thigh2calf: limit (none) -> lower=-2.61 upper=0.0 effort=23.7 velocity=30.0; origin xyz=0 0 -0.214999999999999 rpy=0 -2.139803613507067 0 -> xyz=0 0 -0.214999999999999 rpy=0 0 0; type fixed -> revolute
- joint R_thigh_fix: child rrr_Link -> ru_Link; origin xyz=0.0532497748906444 -0.0144424855132765 0 rpy=0 0 0 -> xyz=0 -0.0577075781855466 0 rpy=0 0 0; parent rr_Link -> rrr_Link

File: bi_urdf/urdf/bi_urdf.urdf (robot description, URDF)
Before this commit: robot bi_urdf, 16 links, 15 joints
Joints:
- removed joint L_base2hip
- removed joint L_calf2wheel
- removed joint L_hip2thigh
- removed joint L_hip_fix
- removed joint L_thigh2calf
- removed joint L_thigh_fix
- removed joint R_base2hip
- removed joint R_calf2wheel
- removed joint R_hip2thigh
- removed joint R_hip_fix
- removed joint R_thigh2calf
- removed joint R_thigh_fix
- added joint l: type continuous, parent base_link, child l_Link, origin xyz=-0.0535148109842794 0.0562499999999701 -0.0547752717334901 rpy=0 0 0, axis 1 0 0
- added joint ld: type continuous, parent lu_Link, child ld_Link, origin xyz=0 0 -0.215 rpy=0 0 0, axis 0 1 0
- added joint ll: type continuous, parent l_Link, child ll_Link, origin xyz=0 0 0 rpy=0 0 0, axis 1 0 0
- added joint lll: type continuous, parent ll_Link, child lll_Link, origin xyz=0.0532497748906447 0.0144424855132758 0 rpy=0 0 0, axis 0 1 0
- added joint lu: type continuous, parent lll_Link, child lu_Link, origin xyz=0 0.0577075781855487 0 rpy=0 0 0, axis 0 1 0
- added joint lw: type continuous, parent ld_Link, child lw_Link, origin xyz=0 0.0286806801421289 -0.215 rpy=0 0 0, axis 0 1 0
- added joint r: type continuous, parent base_link, child r_Link, origin xyz=-0.0535148109842786 -0.0562500000000304 -0.0547752717334899 rpy=0 0 0, axis 1 0 0
- added joint rd: type continuous, parent ru_Link, child rd_Link, origin xyz=0 0 -0.214999999999999 rpy=0 0 0, axis 0 1 0
- added joint rr: type continuous, parent r_Link, child rr_Link, origin xyz=0 0 0 rpy=0 0 0, axis 1 0 0
- added joint rrr: type continuous, parent rr_Link, child rrr_Link, origin xyz=0.0532497748906444 -0.0144424855132765 0 rpy=0 0 0, axis 0 1 0
- added joint ru: type continuous, parent rrr_Link, child ru_Link, origin xyz=0 -0.0577075781855466 0 rpy=0 0 0, axis 0 1 0
- added joint rw: type continuous, parent rd_Link, child rw_Link, origin xyz=0 -0.0286806801421281 -0.215 rpy=0 0 0, axis 0 1 0
- joint bat: type fixed -> continuous
- joint orin: type fixed -> continuous

File: bi_urdf/urdf/bi_urdf_8dof.urdf (robot description, URDF)
Before this commit: robot bi_urdf, 16 links, 15 joints
Links:
- link lw_Link: mass 0.280 -> 0.0
- link rw_Link: mass 0.280 -> 0.0
Joints:
- joint L_base2hip: limit (none) -> lower=0.0 upper=0.0 effort=0.0 velocity=0.0; type fixed -> revolute
- joint L_hip2thigh: child lu_Link -> lll_Link; limit (none) -> lower=0.0 upper=1.57 effort=23.7 velocity=30.0; origin xyz=0 0.0577075781855487 0 rpy=0 1.2164473167519347 0 -> xyz=0.0532497748906447 0.0144424855132758 0 rpy=0 0 0; parent lll_Link -> ll_Link; type fixed -> revolute
- joint L_thigh2calf: limit (none) -> lower=-2.61 upper=0.0 effort=23.7 velocity=30.0; origin xyz=0 0 -0.215 rpy=0 -2.139803613507067 0 -> xyz=0 0 -0.215 rpy=0 0 0; type fixed -> revolute
- joint L_thigh_fix: child lll_Link -> lu_Link; origin xyz=0.0532497748906447 0.0144424855132758 0 rpy=0 0 0 -> xyz=0 0.0577075781855487 0 rpy=0 0 0; parent ll_Link -> lll_Link
- joint R_base2hip: limit (none) -> lower=0.0 upper=0.0 effort=0.0 velocity=0.0; type fixed -> revolute
- joint R_hip2thigh: child ru_Link -> rrr_Link; limit (none) -> lower=0.0 upper=1.57 effort=23.7 velocity=30.0; origin xyz=0 -0.0577075781855466 0 rpy=0 1.2164473167519347 0 -> xyz=0.0532497748906444 -0.0144424855132765 0 rpy=0 0 0; parent rrr_Link -> rr_Link; type fixed -> revolute
- joint R_thigh2calf: limit (none) -> lower=-2.61 upper=0.0 effort=23.7 velocity=30.0; origin xyz=0 0 -0.214999999999999 rpy=0 -2.139803613507067 0 -> xyz=0 0 -0.214999999999999 rpy=0 0 0; type fixed -> revolute
- joint R_thigh_fix: child rrr_Link -> ru_Link; origin xyz=0.0532497748906444 -0.0144424855132765 0 rpy=0 0 0 -> xyz=0 -0.0577075781855466 0 rpy=0 0 0; parent rr_Link -> rrr_Link
